Commit message: Add cartesian controller. Modify for velocity_controller. Add launch file for octmapping

File: xarm_description/urdf/xarm6_with_gripper_realsense.xacro (robot description, xacro)
@@ -6,4 +6,6 @@
   <xacro:arg name="effort_control" default="false"/>
   <xacro:arg name="velocity_control" default="false"/>
+  <xacro:arg name="effort_control_gripper" default="false"/>
+  <xacro:arg name="velocity_control_gripper" default="false"/>
   <!-- load xarm6 robot -->
   <xacro:include filename="$(find xarm_description)/urdf/xarm6_robot_macro.xacro" />
@@ -12,5 +14,5 @@
   <!-- Attach realsense -->
   <xacro:include filename="$(find realsense2_description)/urdf/xarm_d435_camera.urdf.xacro" />
-  <xacro:xarm6_robot prefix="$(arg prefix)" namespace="$(arg ros_namespace)" limited="$(arg limited)" effort_control="$(arg effort_control)" velocity_control="$(arg velocity_control)"/>
-  <xacro:load_gripper attach_to="$(arg prefix)link_eef" effort_control="$(arg effort_control)" velocity_control="$(arg velocity_control)" />
+  <xacro:xarm6_robot prefix="$(arg prefix)" namespace="$(arg ros_namespace)" limited="$(arg limited)" />
+  <xacro:load_gripper attach_to="$(arg prefix)link_eef" />
 </robot>

File: xarm_gripper/urdf/xarm_gripper_model.xacro (robot description, xacro)
@@ -8,9 +8,9 @@
   <xacro:include filename="$(find xarm_gripper)/urdf/xarm_gripper.transmission.xacro" />
   <xacro:include filename="$(find xarm_gripper)/urdf/xarm_gripper.gazebo.xacro" />
-  <xacro:macro name="load_gripper" params="prefix:='' attach_to:='' ns:='xarm' xyz:='0 0 0' rpy:='0 0 0' effort_control:='false' velocity_control:='false' ">
+  <xacro:macro name="load_gripper" params="prefix:='' attach_to:='' ns:='xarm' xyz:='0 0 0' rpy:='0 0 0' effort_control_gripper:='false' velocity_control_gripper:='false' ">
     <!-- gazebo plugin -->
     <!-- <xacro:gazebo_ros_control_plugin namespace="${ns}"/> -->
     <xacro:xarm_gripper_urdf prefix="${prefix}" attach_to="${attach_to}" xyz="${xyz}" rpy="${rpy}" />
-    <xacro:xarm_gripper_transmission prefix="${prefix}" hard_interface="$(eval 'EffortJointInterface' if effort_control else 'VelocityJointInterface' if velocity_control else 'PositionJointInterface')" />
+    <xacro:xarm_gripper_transmission prefix="${prefix}" hard_interface="$(eval 'EffortJointInterface' if effort_control_gripper else 'VelocityJointInterface' if velocity_control_gripper else 'PositionJointInterface')" />
     <xacro:xarm_gripper_gazebo prefix="${prefix}" />
     <!-- mimic_joint_plugin has to be installed: -->

Commit message: Change method for attaching realsense to xarm.

File: xarm_description/urdf/xarm6_with_gripper_realsense.xacro (robot description, xacro)
@@ -8,4 +8,10 @@
   <xacro:arg name="effort_control_gripper" default="false"/>
   <xacro:arg name="velocity_control_gripper" default="false"/>
+  <!-- For d435 -->
+  <xacro:arg name="use_nominal_extrinsics" default="false"/>
+  <xacro:arg name="add_plug" default="false" />
+  <xacro:arg name="use_mesh" default="true" />
+  <xacro:arg name="topics_ns" default="camera" />
+  <xacro:arg name="publish_pointcloud" default="true" />
   <!-- load xarm6 robot -->
   <xacro:include filename="$(find xarm_description)/urdf/xarm6_robot_macro.xacro" />
@@ -13,6 +19,9 @@
   <xacro:include filename="$(find xarm_gripper)/urdf/xarm_gripper_model.xacro" />
   <!-- Attach realsense -->
-  <xacro:include filename="$(find realsense2_description)/urdf/xarm_d435_camera.urdf.xacro" />
+  <xacro:include filename="$(find realsense2_description)/urdf/_d435.urdf.xacro" />
   <xacro:xarm6_robot prefix="$(arg prefix)" namespace="$(arg ros_namespace)" limited="$(arg limited)" />
   <xacro:load_gripper attach_to="$(arg prefix)link_eef" />
+  <xacro:sensor_d435 parent="$(arg prefix)link_eef" use_nominal_extrinsics="$(arg use_nominal_extrinsics)" add_plug="$(arg add_plug)" use_mesh="$(arg use_mesh)" topics_ns="$(arg topics_ns)" publish_pointcloud="$(arg publish_pointcloud)" >
+    <origin xyz="0.055 0 0.012" rpy="0 ${-pi/2} ${pi}"/>
+  </xacro:sensor_d435>
 </robot>
